Commit message: Replace the UR URDF

File: ur_description/urdf/ur_macro.xacro (robot description, xacro)
@@ -63,46 +63,43 @@
     <!-- Add URDF transmission elements (for ros_control) -->
     <xacro:ur_arm_transmission prefix="${prefix}" hw_interface="${transmission_hw_interface}" />
-    <!-- main serial chain -->
     <link
       name="${prefix}base_link">
       <inertial>
         <origin
-          xyz="0 0 0.014753"
-          rpy="0 0 0" />
-        <mass
-          value="0.82586" />
-        <inertia
-          ixx="0.0020803"
-          ixy="1.735E-19"
-          ixz="3.2973E-19"
-          iyy="0.0020803"
-          iyz="3.6808E-19"
-          izz="0.0039193" />
-      </inertial>
-      <visual>
-        <origin
-          xyz="0 0 0"
-          rpy="0 0 0" />
-        <geometry>
-          <mesh
-            filename="package://al_arm_5_2/meshes/base.STL" />
-        </geometry>
-        <material
-          name="">
-          <color
-            rgba="0.79216 0.81961 0.93333 1" />
-        </material>
-      </visual>
-<!--
-      <collision>
-        <origin
-          xyz="0 0 0"
-          rpy="0 0 0" />
-        <geometry>
-          <mesh
-            filename="package://al_arm_5_2/meshes/base.STL" />
-        </geometry>
-      </collision>
--->
+          xyz="-6.93889390390723E-18 2.77555756156289E-17 0.0147527451068121"
+          rpy="0 0 0" />
+        <mass
+          value="0.825861073097743" />
+        <inertia
+          ixx="0.00208027891140234"
+          ixy="-7.14684049245823E-19"
+          ixz="4.50656009154085E-19"
+          iyy="0.00208027891140235"
+          iyz="-5.57841619598388E-19"
+          izz="0.00391932737987958" />
+      </inertial>
+      <visual>
+        <origin
+          xyz="0 0 0"
+          rpy="0 0 0" />
+        <geometry>
+          <mesh
+            filename="package://al_arm_2_3_t1/meshes/Base.STL" />
+        </geometry>
+        <material
+          name="">
+          <color
+            rgba="0.792156862745098 0.819607843137255 0.933333333333333 1" />
+        </material>
+      </visual>
+      <collision>
+        <origin
+          xyz="0 0 0"
+          rpy="0 0 0" />
+        <geometry>
+          <mesh
+            filename="package://al_arm_2_3_t1/meshes/Base.STL" />
+        </geometry>
+      </collision>
     </link>
     <link
@@ -110,41 +107,39 @@
       <inertial>
         <origin
-          xyz="0.0057811 -4.7696E-10 0.086487"
-          rpy="0 0 3.141" />
-        <mass
-          value="2.207" />
-        <inertia
-          ixx="0.0095841"
-          ixy="8.9967E-10"
-          ixz="-0.0003"
-          iyy="0.0097275"
-          iyz="4.4737E-10"
-          izz="0.0055768" />
-      </inertial>
-      <visual>
-        <origin
-          xyz="0 0 0"
-          rpy="0 0 3.141" />
-        <geometry>
-          <mesh
-            filename="package://al_arm_5_2/meshes/seg1.STL" />
-        </geometry>
-        <material
-          name="">
-          <color
-            rgba="0.50196 0.50196 1 1" />
-        </material>
-      </visual>
-<!--
-      <collision>
-        <origin
-          xyz="0 0 0"
-          rpy="0 0 0" />
-        <geometry>
-          <mesh
-            filename="package://al_arm_5_2/meshes/seg1.STL" />
-        </geometry>
-      </collision>
--->
+          xyz="0.00578107509486808 -4.76958778028447E-10 0.0864872761296608"
+          rpy="0 0 3.1415" />
+        <mass
+          value="2.20704513466782" />
+        <inertia
+          ixx="0.00958414619563909"
+          ixy="8.99674275410972E-10"
+          ixz="-0.000299996856367022"
+          iyy="0.00972749157915772"
+          iyz="4.47374741596083E-10"
+          izz="0.00557677453899358" />
+      </inertial>
+      <visual>
+        <origin
+          xyz="0 0 0"
+          rpy="0 0 0" />
+        <geometry>
+          <mesh
+            filename="package://al_arm_2_3_t1/meshes/Seg1.STL" />
+        </geometry>
+        <material
+          name="">
+          <color
+            rgba="0.501960784313725 0.501960784313725 1 1" />
+        </material>
+      </visual>
+      <collision>
+        <origin
+          xyz="0 0 0"
+          rpy="0 0 0" />
+        <geometry>
+          <mesh
+            filename="package://al_arm_2_3_t1/meshes/Seg1.STL" />
+        </geometry>
+      </collision>
     </link>
     <joint
@@ -153,5 +148,5 @@
       <origin
         xyz="0 0 0.0427"
-        rpy="0 0 ${pi/2}" />
+        rpy="0 0 0" />
       <parent link="${prefix}base_link" />
       <child link="${prefix}shoulder_link" />
@@ -159,6 +154,6 @@
         xyz="0 0 1" />
       <limit
-        lower="-3.14"
-        upper="3.14"
+        lower="-1.571"
+        upper="1.571"
         effort="0"
         velocity="0" />
@@ -168,41 +163,39 @@
       <inertial>
         <origin
-          xyz="0.6 0.0005672 0.085941"
-          rpy="0 0 0" />
-        <mass
-          value="2.1" />
-        <inertia
-          ixx="0.0096686"
-          ixy="-1.7798E-05"
-          ixz="-2.2764E-05"
-          iyy="0.0097485"
-          iyz="-4.8304E-06"
-          izz="0.0051536" />
-      </inertial>
-      <visual>
-        <origin
-          xyz="0 0 0"
-          rpy="0 0 0" />
-        <geometry>
-          <mesh
-            filename="package://al_arm_5_2/meshes/seg2.STL" />
-        </geometry>
-        <material
-          name="">
-          <color
-            rgba="0.50196 0.50196 1 1" />
-        </material>
-      </visual>
-<!--
-      <collision>
-        <origin
-          xyz="0 0 0"
-          rpy="0 0 0" />
-        <geometry>
-          <mesh
-            filename="package://al_arm_5_2/meshes/seg2.STL" />
-        </geometry>
-      </collision>
--->
+          xyz="0.00236385799568389 0.00136442528422548 0.145940570815008"
+          rpy="0 0 0" />
+        <mass
+          value="2.10002062392676" />
+        <inertia
+          ixx="0.0096866811667758"
+          ixy="-3.78905636830833E-05"
+          ixz="-2.01582616482002E-05"
+          iyy="0.00973042156076894"
+          iyz="-1.16285177834027E-05"
+          izz="0.0051535893543322" />
+      </inertial>
+      <visual>
+        <origin
+          xyz="0 0 0"
+          rpy="0 0 0" />
+        <geometry>
+          <mesh
+            filename="package://al_arm_2_3_t1/meshes/Seg2.STL" />
+        </geometry>
+        <material
+          name="">
+          <color
+            rgba="0.501960784313725 0.501960784313725 1 1" />
+        </material>
+      </visual>
+      <collision>
+        <origin
+          xyz="0 0 0"
+          rpy="0 0 0" />
+        <geometry>
+          <mesh
+            filename="package://al_arm_2_3_t1/meshes/Seg2.STL" />
+        </geometry>
+      </collision>
     </link>
     <joint
@@ -210,6 +203,6 @@
       type="revolute">
       <origin
-        xyz="-0.06 0 0.11"
-        rpy="0 -1.5708 0" />
+        xyz="0 0 0.11"
+        rpy="3.1415 -1.5708 0" />
       <parent link="${prefix}shoulder_link" />
       <child link="${prefix}upper_arm_link" />
@@ -217,6 +210,6 @@
         xyz="0 0 1" />
       <limit
-        lower="-3.14"
-        upper="3.14"
+        lower="-1.571"
+        upper="1.571"
         effort="0"
         velocity="0" />
@@ -226,41 +219,90 @@
       <inertial>
         <origin
-          xyz="-5.0864E-07 0.0083839 0.20092"
-          rpy="0 0 0" />
-        <mass
-          value="0.81968" />
-        <inertia
-          ixx="0.0025453"
-          ixy="-5.2922E-10"
-          ixz="-3.0369E-10"
-          iyy="0.0016077"
-          iyz="-0.00011692"
-          izz="0.0019806" />
-      </inertial>
-      <visual>
-        <origin
-          xyz="0 0 0"
-          rpy="0 0 0" />
-        <geometry>
-          <mesh
-            filename="package://al_arm_5_2/meshes/seg3.STL" />
-        </geometry>
-        <material
-          name="">
-          <color
-            rgba="0.89804 0.91765 0.92941 1" />
-        </material>
-      </visual>
-<!--
-      <collision>
-        <origin
-          xyz="0 0 0"
-          rpy="0 0 0" />
-        <geometry>
-          <mesh
-            filename="package://al_arm_5_2/meshes/seg3.STL" />
-        </geometry>
-      </collision>
--->
+          xyz="-0.00838393613902233 -4.91095186582607E-07 0.260922409686664"
+          rpy="0 0 0" />
+        <mass
+          value="0.819681577987536" />
+        <inertia
+          ixx="0.00160765831987408"
+          ixy="5.92417274710161E-10"
+          ixz="0.000116924443578868"
+          iyy="0.00254525158547177"
+          iyz="-2.77379135949023E-10"
+          izz="0.00198059878006" />
+      </inertial>
+      <visual>
+        <origin
+          xyz="0 0 0"
+          rpy="0 0 0" />
+        <geometry>
+          <mesh
+            filename="package://al_arm_2_3_t1/meshes/Seg3.STL" />
+        </geometry>
+        <material
+          name="">
+          <color
+            rgba="0.898039215686275 0.917647058823529 0.929411764705882 1" />
+        </material>
+      </visual>
+      <collision>
+        <origin
+          xyz="0 0 0"
+          rpy="0 0 0" />
+        <geometry>
+          <mesh
+            filename="package://al_arm_2_3_t1/meshes/Seg3.STL" />
+        </geometry>
+      </collision>
+    </link>
+    <joint
+      name="Joint_2"
+      type="fixed">
+      <origin
+        xyz="0 0 0.15"
+        rpy="0.5236 -1.5708 3.1415" />
+      <parent
+        link="${prefix}upper_arm_link" />
+      <child
+        link="${prefix}forearm_link" />
+    </joint>
+    <link
+      name="${prefix}wrist_1_link">
+      <inertial>
+        <origin
+          xyz="-0.0144066128415552 -0.00831766306521403 0.138440702841905"
+          rpy="0 0 0" />
+        <mass
+          value="1.19693957833335" />
+        <inertia
+          ixx="0.00146338839182427"
+          ixy="-7.75815880987421E-05"
+          ixz="0.000235267465053867"
+          iyy="0.00155297172259349"
+          iyz="0.000135831693069045"
+          izz="0.00142951512500459" />
+      </inertial>
+      <visual>
+        <origin
+          xyz="0 0 0"
+          rpy="0 0 0.53" />
+        <geometry>
+          <mesh
+            filename="package://al_arm_2_3_t1/meshes/Seg4.STL" />
+        </geometry>
+        <material
+          name="">
+          <color
+            rgba="0.501960784313725 0.501960784313725 1 1" />
+        </material>
+      </visual>
+      <collision>
+        <origin
+          xyz="0 0 0"
+          rpy="0 0 0" />
+        <geometry>
+          <mesh
+            filename="package://al_arm_2_3_t1/meshes/Seg4.STL" />
+        </geometry>
+      </collision>
     </link>
     <joint
@@ -268,71 +310,13 @@
       type="revolute">
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
Commit message: The robot moves! TCP needs adjustment, though

File: ur_description/urdf/ur_macro.xacro (robot description, xacro)
@@ -93,4 +93,5 @@
         </material>
       </visual>
+<!--
       <collision>
         <origin
@@ -102,4 +103,5 @@
         </geometry>
       </collision>
+-->
     </link>
     <link
@@ -133,4 +135,5 @@
         </material>
       </visual>
+<!--
       <collision>
         <origin
@@ -142,4 +145,5 @@
         </geometry>
       </collision>
+-->
     </link>
     <joint
@@ -189,4 +193,5 @@
         </material>
       </visual>
+<!--
       <collision>
         <origin
@@ -198,4 +203,5 @@
         </geometry>
       </collision>
+-->
     </link>
     <joint
@@ -245,4 +251,5 @@
         </material>
       </visual>
+<!--
       <collision>
         <origin
@@ -254,4 +261,5 @@
         </geometry>
       </collision>
+-->
     </link>
     <joint
@@ -296,4 +304,5 @@
         </material>
       </visual>
+<!--
       <collision>
         <origin
@@ -305,4 +314,5 @@
         </geometry>
       </collision>
+-->
     </link>
     <joint
@@ -352,4 +362,5 @@
         </material>
       </visual>
+<!--
       <collision>
         <origin
@@ -361,4 +372,5 @@
         </geometry>
       </collision>
+-->
     </link>
     <joint
@@ -408,4 +420,5 @@
         </material>
       </visual>
+<!--
       <collision>
         <origin
@@ -417,4 +430,5 @@
         </geometry>
       </collision>
+-->
     </link>
     <joint
@@ -464,4 +478,5 @@
         </material>
       </visual>
+<!--
       <collision>
         <origin
@@ -473,4 +488,5 @@
         </geometry>
       </collision>
+-->
     </link>
     <joint
@@ -516,5 +532,5 @@
       <!-- default toolframe: X+ left, Y+ up, Z+ front -->
       <origin xyz="0 0 0" rpy="${pi/2.0} 0 ${pi/2.0}"/>
-      <parent link="${prefix}flange"/>
+      <parent link="${prefix}EOAT"/>
       <child link="${prefix}tool0"/>
     </joint>

Commit message: Fix joint locations in ur_macro.xacro

File: ur_description/urdf/ur_macro.xacro (robot description, xacro)
@@ -106,5 +106,5 @@
     </link>
     <link
-      name="${prefix}shoulder_link">
+      name="${prefix}Seg1">
       <inertial>
         <origin
@@ -153,16 +153,18 @@
         xyz="0 0 0.0427"
         rpy="0 0 0" />
-      <parent link="${prefix}base_link" />
-      <child link="${prefix}shoulder_link" />
+      <parent
+        link="base_link" />
+      <child
+        link="Seg1" />
       <axis
         xyz="0 0 1" />
       <limit
-        lower="-3.14"
-        upper="3.14"
+        lower="-3.14159"
+        upper="3.14159"
         effort="0"
         velocity="0" />
     </joint>
     <link
-      name="${prefix}upper_arm_link">
+      name="${prefix}Seg2">
       <inertial>
         <origin
@@ -211,16 +213,18 @@
         xyz="0 0 0.11"
         rpy="3.1415 -1.5708 0" />
-      <parent link="${prefix}shoulder_link" />
-      <child link="${prefix}upper_arm_link" />
+      <parent
+        link="Seg1" />
+      <child
+        link="Seg2" />
       <axis
         xyz="0 0 1" />
       <limit
-        lower="-3.14"
-        upper="3.14"
+        lower="-3.14159"
+        upper="3.14159"
         effort="0"
         velocity="0" />
     </joint>
     <link
-      name="${prefix}forearm_link">
+      name="${prefix}Seg3">
       <inertial>
         <origin
@@ -264,5 +268,5 @@
     </link>
     <joint
-      name="Joint_2"
+      name="${prefix}Joint_2"
       type="fixed">
       <origin
@@ -270,10 +274,10 @@
         rpy="0.5236 -1.5708 3.1415" />
       <parent
-        link="${prefix}upper_arm_link" />
-      <child
-        link="${prefix}forearm_link" />
-    </joint>
-    <link
-      name="${prefix}wrist_1_link">
+        link="Seg2" />
+      <child
+        link="Seg3" />
+    </joint>
+    <link
+      name="${prefix}Seg4">
       <inertial>
         <origin
@@ -322,16 +326,18 @@
         xyz="0 0 0.304"
         rpy="3.1416 -1.5708 3.1416" />
-      <parent link="${prefix}forearm_link" />
-      <child link="${prefix}wrist_1_link" />
+      <parent
+        link="Seg3" />
+      <child
+        link="Seg4" />
       <axis
         xyz="0 0 -1" />
       <limit
-        lower="-3.14"
-        upper="3.14"
+        lower="-3.14159"
+        upper="3.14159"
         effort="0"
         velocity="0" />
     </joint>
     <link
-      name="${prefix}wrist_2_link">
+      name="${prefix}Seg5">
       <inertial>
         <origin
@@ -375,25 +381,60 @@
     </link>
     <joint
+      name="${prefix}Joint_4"
+      type="fixed">
+      <origin
+        xyz="0 0 0.15013"
+        rpy="2.618 -1.5708 -1.5708" />
+      <parent
+        link="Seg4" />
+      <child
+        link="Seg5" />
+    </joint>
+    <joint
       name="${prefix}wrist_1_joint"
       type="revolute">
       <origin
-        xyz="0 0 0.15013"
-        rpy="2.618 -1.5708 -1.5708" />
-      <parent link="${prefix}wrist_1_link" />
-      <child link="${prefix}wrist_2_link" />
+        xyz="0 0 0.1802"
+        rpy="0 -1.5708 3.1416" />
+      <parent
+        link="Seg5" />
+      <child
+        link="J5InvisibleLink" />
       <axis
         xyz="0 0 -1" />
       <limit
-        lower="-3.14"
-        upper="3.14"
+        lower="-3.14159"
+        upper="3.14159"
         effort="0"
         velocity="0" />
     </joint>
-    <link
-      name="${prefix}wrist_3_link">
-      <inertial>
-        <origin
-          xyz="0.00221631980461306 -0.00682201775014385 0.0998520497439655"
-          rpy="0 0 0" />
+    <!-- The meshes for this link weren't exported right, so it has invisible links -->
+    <link
+      name="${prefix}J5InvisibleLink">
+    </link>
+    <joint
+      name="${prefix}wrist_2_joint"
+      type="revolute">
+      <origin
+        xyz="0 0 0.12"
+        rpy="0 0 0" />
+      <parent
+        link="J5InvisibleLink" />
+      <child
+        link="Seg6" />
+      <axis
+        xyz="0 1 0" />
+      <limit
+        lower="-3.14159"
+        upper="3.14159"
+        effort="0"
+        velocity="0" />
+    </joint>
+    <link
+      name="${prefix}Seg6">
+      <inertial>
+        <origin
+          xyz="0 0 -0.12"
+          rpy="0 0 -0.3" />
         <mass
           value="0.719205488845403" />
@@ -406,8 +447,9 @@
           izz="0.00177485843278574" />
       </inertial>
-      <visual>
-        <origin
-          xyz="0 0 0"
-          rpy="0 0 0" />
+  <!--
+      <visual>
+        <origin
+          xyz="0 0 -0.12"
+          rpy="0 0 -0.3" />
         <geometry>
           <mesh
@@ -420,9 +462,8 @@
         </material>
       </visual>
-<!--
-      <collision>
-        <origin
-          xyz="0 0 0"
-          rpy="0 0 0" />
+      <collision>
+        <origin
+          xyz="0 0 -0.12"
+          rpy="0 0 -0.3" />
         <geometry>
           <mesh
@@ -430,28 +471,12 @@
         </geometry>
       </collision>
--->
-    </link>
-    <joint
-      name="${prefix}wrist_2_joint"
-      type="revolute">
-      <origin
-        xyz="0 0 0.1802"
-        rpy="0 -1.5708 3.1416" />
-      <parent link="${prefix}wrist_2_link" />
-      <child link="${prefix}wrist_3_link" />
-      <axis
-        xyz="0 0 -1" />
-      <limit
-        lower="-3.14"
-        upper="3.14"
-        effort="0"
-        velocity="0" />
-    </joint>
-    <link
-      name="EOAT">
+  -->
+    </link>
+    <link
+      name="${prefix}EOAT">
       <inertial>
         <origin
           xyz="-2.38657933762654E-07 0.0813741192774262 0.108881870556287"
-          rpy="0 0 0" />
+          rpy="-1.571 -1.571 1.571" />
         <mass
           value="1.78761153567891" />
@@ -466,6 +491,6 @@
       <visual>
         <origin
-          xyz="0 0 -0.12"
-          rpy="0 0 0" />
+          xyz="0.12 0 0"
+          rpy="-1.571 -1.571 1.571" />
         <geometry>
           <mesh
@@ -481,6 +506,6 @@
       <collision>
         <origin
-          xyz="0 0 -0.12"
-          rpy="0 0 0" />
+          xyz="0.12 0 0"
+          rpy="-1.571 -1.571 1.571" />
         <geometry>
           <mesh
@@ -494,8 +519,8 @@
       type="revolute">
       <origin
-        xyz="-0.02 0.1 0.12"
-        rpy="1.885 -1.5708 3.1416" />
-      <parent
-        link="${prefix}wrist_3_link" />
+        xyz="0 0.12 0"
+        rpy="0 0 -1.5708" />
+      <parent
+        link="Seg6" />
       <child
         link="EOAT" />
@@ -503,6 +528,6 @@
         xyz="0 1 0" />
       <limit
-        lower="-3.14"
-        upper="3.14"
+        lower="-3.14159"
+        upper="3.14159"
         effort="0"
         velocity="0" />
@@ -523,5 +548,5 @@
     <link name="${prefix}flange" />
     <joint name="${prefix}wrist_3-flange" type="fixed">
-      <parent link="${prefix}wrist_3_link" />
+      <parent link="${prefix}Seg6" />
       <child link="${prefix}flange" />
       <origin xyz="0 0 0" rpy="0 ${-pi/2.0} ${-pi/2.0}" />
