Commit message: The URDF loads

File: ur_description/urdf/ur_macro.xacro (robot description, xacro)
@@ -66,143 +66,275 @@
     <link name="${prefix}base_link"/>
     <link name="${prefix}base_link_inertia">
-      <visual>
-        <origin xyz="0 0 0" rpy="0 0 ${pi}"/>
-        <geometry>
-          <mesh filename="${base_visual_mesh}"/>
-        </geometry>
-        <material name="${base_visual_material_name}">
-          <color rgba="${base_visual_material_color}"/>
-        </material>
-      </visual>
-      <collision>
-        <origin xyz="0 0 0" rpy="0 0 ${pi}"/>
-        <geometry>
-          <mesh filename="${base_collision_mesh}"/>
-        </geometry>
-      </collision>
-      <xacro:cylinder_inertial radius="${base_inertia_radius}" length="${base_inertia_length}" mass="${base_mass}">
-        <origin xyz="0 0 0" rpy="0 0 0" />
-      </xacro:cylinder_inertial>
+      <inertial>
+        <origin
+          xyz="0 0 0.014753"
+          rpy="0 0 0" />
+        <mass
+          value="0.82586" />
+        <inertia
+          ixx="0.0020803"
+          ixy="1.735E-19"
+          ixz="3.2973E-19"
+          iyy="0.0020803"
+          iyz="3.6808E-19"
+          izz="0.0039193" />
+      </inertial>
+      <visual>
+        <origin
+          xyz="0 0 0"
+          rpy="0 0 0" />
+        <geometry>
+          <mesh
+            filename="package://al_arm_5_2/meshes/base.STL" />
+        </geometry>
+        <material
+          name="">
+          <color
+            rgba="0.79216 0.81961 0.93333 1" />
+        </material>
+      </visual>
+      <collision>
+        <origin
+          xyz="0 0 0"
+          rpy="0 0 0" />
+        <geometry>
+          <mesh
+            filename="package://al_arm_5_2/meshes/base.STL" />
+        </geometry>
+      </collision>
     </link>
     <link name="${prefix}shoulder_link">
-      <visual>
-        <origin xyz="0 0 0" rpy="0 0 ${pi}"/>
-        <geometry>
-          <mesh filename="${shoulder_visual_mesh}"/>
-        </geometry>
-        <material name="${shoulder_visual_material_name}">
-          <color rgba="${shoulder_visual_material_color}"/>
-        </material>
-      </visual>
-      <collision>
-        <origin xyz="0 0 0" rpy="0 0 ${pi}"/>
-        <geometry>
-          <mesh filename="${shoulder_collision_mesh}"/>
-        </geometry>
-      </collision>
-      <xacro:cylinder_inertial radius="${shoulder_inertia_radius}" length="${shoulder_inertia_length}" mass="${shoulder_mass}">
-        <origin xyz="0 0 0" rpy="0 0 0" />
-      </xacro:cylinder_inertial>
+      <inertial>
+        <origin
+          xyz="0.0057811 -4.7696E-10 0.086487"
+          rpy="0 0 3.141" />
+        <mass
+          value="2.207" />
+        <inertia
+          ixx="0.0095841"
+          ixy="8.9967E-10"
+          ixz="-0.0003"
+          iyy="0.0097275"
+          iyz="4.4737E-10"
+          izz="0.0055768" />
+      </inertial>
+      <visual>
+        <origin
+          xyz="0 0 0"
+          rpy="0 0 3.141" />
+        <geometry>
+          <mesh
+            filename="package://al_arm_5_2/meshes/seg1.STL" />
+        </geometry>
+        <material
+          name="">
+          <color
+            rgba="0.50196 0.50196 1 1" />
+        </material>
+      </visual>
+      <collision>
+        <origin
+          xyz="0 0 0"
+          rpy="0 0 0" />
+        <geometry>
+          <mesh
+            filename="package://al_arm_5_2/meshes/seg1.STL" />
+        </geometry>
+      </collision>
     </link>
     <link name="${prefix}upper_arm_link">
-      <visual>
-        <origin xyz="0 0 ${shoulder_offset}" rpy="${pi/2} 0 ${-pi/2}"/>
-        <geometry>
-          <mesh filename="${upper_arm_visual_mesh}"/>
-        </geometry>
-        <material name="${upper_arm_visual_material_name}">
-          <color rgba="${upper_arm_visual_material_color}"/>
-        </material>
-      </visual>
-      <collision>
-        <origin xyz="0 0 ${shoulder_offset}" rpy="${pi/2} 0 ${-pi/2}"/>
-        <geometry>
-          <mesh filename="${upper_arm_collision_mesh}"/>
-        </geometry>
-      </collision>
-      <xacro:cylinder_inertial radius="${upperarm_inertia_radius}" length="${upperarm_inertia_length}" mass="${upper_arm_mass}">
-        <origin xyz="${-0.5 * upperarm_inertia_length} 0.0 ${upper_arm_inertia_offset}" rpy="0 ${pi/2} 0" />
-      </xacro:cylinder_inertial>
+      <inertial>
+        <origin
+          xyz="0.6 0.0005672 0.085941"
+          rpy="0 0 0" />
+        <mass
+          value="2.1" />
+        <inertia
+          ixx="0.0096686"
+          ixy="-1.7798E-05"
+          ixz="-2.2764E-05"
+          iyy="0.0097485"
+          iyz="-4.8304E-06"
+          izz="0.0051536" />
+      </inertial>
+      <visual>
+        <origin
+          xyz="0 0 0"
+          rpy="0 0 0" />
+        <geometry>
+          <mesh
+            filename="package://al_arm_5_2/meshes/seg2.STL" />
+        </geometry>
+        <material
+          name="">
+          <color
+            rgba="0.50196 0.50196 1 1" />
+        </material>
+      </visual>
+      <collision>
+        <origin
+          xyz="0 0 0"
+          rpy="0 0 0" />
+        <geometry>
+          <mesh
+            filename="package://al_arm_5_2/meshes/seg2.STL" />
+        </geometry>
+      </collision>
     </link>
     <link name="${prefix}forearm_link">
-      <visual>
-        <origin xyz="0 0 ${elbow_offset}" rpy="${pi/2} 0 ${-pi/2}"/>
-        <geometry>
-          <mesh filename="${forearm_visual_mesh}"/>
-        </geometry>
-        <material name="${forearm_visual_material_name}">
-          <color rgba="${forearm_visual_material_color}"/>
-        </material>
-      </visual>
-      <collision>
-        <origin xyz="0 0 ${elbow_offset}" rpy="${pi/2} 0 ${-pi/2}"/>
-        <geometry>
-          <mesh filename="${forearm_collision_mesh}"/>
-        </geometry>
-      </collision>
-      <xacro:cylinder_inertial radius="${forearm_inertia_radius}" length="${forearm_inertia_length}"  mass="${forearm_mass}">
-        <origin xyz="${-0.5 * forearm_inertia_length} 0.0 ${elbow_offset}" rpy="0 ${pi/2} 0" />
-      </xacro:cylinder_inertial>
+      <inertial>
+        <origin
+          xyz="-5.0864E-07 0.0083839 0.20092"
+          rpy="0 0 0" />
+        <mass
+          value="0.81968" />
+        <inertia
+          ixx="0.0025453"
+          ixy="-5.2922E-10"
+          ixz="-3.0369E-10"
+          iyy="0.0016077"
+          iyz="-0.00011692"
+          izz="0.0019806" />
+      </inertial>
+      <visual>
+        <origin
+          xyz="0 0 0"
+          rpy="0 0 0" />
+        <geometry>
+          <mesh
+            filename="package://al_arm_5_2/meshes/seg3.STL" />
+        </geometry>
+        <material
+          name="">
+          <color
+            rgba="0.89804 0.91765 0.92941 1" />
+        </material>
+      </visual>
+      <collision>
+        <origin
+          xyz="0 0 0"
+          rpy="0 0 0" />
+        <geometry>
+          <mesh
+            filename="package://al_arm_5_2/meshes/seg3.STL" />
+        </geometry>
+      </collision>
     </link>
     <link name="${prefix}wrist_1_link">
-      <visual>
-        <!-- TODO: Move this to a parameter -->
-        <origin xyz="0 0 ${wrist_1_visual_offset}" rpy="${pi/2} 0 0"/>
-        <geometry>
-          <mesh filename="${wrist_1_visual_mesh}"/>
-        </geometry>
-        <material name="${wrist_1_visual_material_name}">
-          <color rgba="${wrist_1_visual_material_color}"/>
-        </material>
-      </visual>
-      <collision>
-        <origin xyz="0 0 ${wrist_1_visual_offset}" rpy="${pi/2} 0 0"/>
-        <geometry>
-          <mesh filename="${wrist_1_collision_mesh}"/>
-        </geometry>
-      </collision>
-      <xacro:cylinder_inertial radius="${wrist_1_inertia_radius}" length="${wrist_1_inertia_length}"  mass="${wrist_1_mass}">
-        <origin xyz="0 0 0" rpy="0 0 0" />
-      </xacro:cylinder_inertial>
+      <inertial>
+        <origin
+          xyz="0.028904 -0.03325 0.050924"
+          rpy="0 0 0" />
+        <mass
+          value="1.5416" />
+        <inertia
+          ixx="0.0025041"
+          ixy="0.00055564"
+          ixz="-0.00017823"
+          iyy="0.0023479"
+          iyz="0.00020503"
+          izz="0.0028189" />
+      </inertial>
+      <visual>
+        <origin
+          xyz="0 0 0"
+          rpy="0 0 0" />
+        <geometry>
+          <mesh
+            filename="package://al_arm_5_2/meshes/seg4.STL" />
+        </geometry>
+        <material
+          name="">
+          <color
+            rgba="0.50196 0.50196 1 1" />
+        </material>
+      </visual>
+      <collision>
+        <origin
+          xyz="0 0 0"
+          rpy="0 0 0" />
+        <geometry>
+          <mesh
+            filename="package://al_arm_5_2/meshes/seg4.STL" />
+        </geometry>
+      </collision>
     </link>
     <link name="${prefix}wrist_2_link">
-      <visual>
-        <origin xyz="0 0 ${wrist_2_visual_offset}" rpy="0 0 0"/>
-        <geometry>
-          <mesh filename="${wrist_2_visual_mesh}"/>
-        </geometry>
-        <material name="${wrist_2_visual_material_name}">
-          <color rgba="${wrist_2_visual_material_color}"/>
-        </material>
-      </visual>
-      <collision>
-        <origin xyz="0 0 ${wrist_2_visual_offset}" rpy="0 0 0"/>
-        <geometry>
-          <mesh filename="${wrist_2_collision_mesh}"/>
-        </geometry>
-      </collision>
-      <xacro:cylinder_inertial radius="${wrist_2_inertia_radius}" length="${wrist_2_inertia_length}"  mass="${wrist_2_mass}">
-        <origin xyz="0 0 0" rpy="0 0 0" />
-      </xacro:cylinder_inertial>
+      <inertial>
+        <origin
+          xyz="5.2201E-07 -0.003931 0.039853"
+          rpy="0 0 0" />
+        <mass
+          value="0.71921" />
+        <inertia
+          ixx="0.0019666"
+          ixy="-3.0762E-10"
+          ixz="1.656E-11"
+          iyy="0.0010669"
+          iyz="5.6958E-05"
+          izz="0.0017541" />
+      </inertial>
+      <visual>
+        <origin
+          xyz="0 0 0"
+          rpy="0 0 0" />
+        <geometry>
+          <mesh
+            filename="package://al_arm_5_2/meshes/seg5.STL" />
+        </geometry>
+        <material
+          name="">
+          <color
+            rgba="0.50196 0.50196 1 1" />
+        </material>
+      </visual>
+      <collision>
+        <origin
+          xyz="0 0 0"
+          rpy="0 0 0" />
+        <geometry>
+          <mesh
+            filename="package://al_arm_5_2/meshes/seg5.STL" />
+        </geometry>
+      </collision>
     </link>
     <link name="${prefix}wrist_3_link">
-      <visual>
-        <origin xyz="0 0 ${wrist_3_visual_offset}" rpy="${pi/2} 0 0"/>
-        <geometry>
-          <mesh filename="${wrist_3_visual_mesh}"/>
-        </geometry>
-        <material name="${wrist_3_visual_material_name}">
-          <color rgba="${wrist_3_visual_material_color}"/>
-        </material>
-      </visual>
-      <collision>
-        <origin xyz="0 0 ${wrist_3_visual_offset}" rpy="${pi/2} 0 0"/>
-        <geometry>
-          <mesh filename="${wrist_3_collision_mesh}"/>
-        </geometry>
-      </collision>
-      <xacro:cylinder_inertial radius="${wrist_3_inertia_radius}" length="${wrist_3_inertia_length}"  mass="${wrist_3_mass}">
-        <origin xyz="0.0 0.0 ${-0.5 * wrist_3_inertia_length}" rpy="0 0 0" />
-      </xacro:cylinder_inertial>
+      <inertial>
+        <origin
+          xyz="-0.0030119 -0.097795 0.051894"
+          rpy="0 0 0" />
+        <mass
+          value="1.7876" />
+        <inertia
+          ixx="0.0067992"
+          ixy="0.00061613"
+          ixz="8.5775E-11"
+          iyy="0.0022268"
+          iyz="5.6958E-05"
+          izz="0.006937" />
+      </inertial>
+      <visual>
+        <origin
+          xyz="0 0 -0.06"
+          rpy="0 0 0" />
+        <geometry>
+          <mesh
+            filename="package://al_arm_5_2/meshes/seg6.STL" />
+        </geometry>
+        <material
+          name="">
+          <color
+            rgba="0.50196 0.50196 1 1" />
+        </material>
+      </visual>
+      <collision>
+        <origin
+          xyz="0 0 -0.06"
+          rpy="0 0 0" />
+        <geometry>
+          <mesh
+            filename="package://al_arm_5_2/meshes/seg6.STL" />
+        </geometry>
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
Commit message: Correct tool0, wider joint limits

File: ur_description/urdf/ur_macro.xacro (robot description, xacro)
@@ -372,6 +372,6 @@
         xyz="0 0 1" />
       <limit
-        lower="-3.14"
-        upper="3.14"
+        lower="-6.28"
+        upper="6.28"
         effort="0"
         velocity="0" />
@@ -386,6 +386,6 @@
         xyz="0 0 1" />
       <limit
-        lower="-3.14"
-        upper="3.14"
+        lower="-6.28"
+        upper="6.28"
         effort="0"
         velocity="0" />
@@ -398,6 +398,6 @@
       <child link="${prefix}forearm_link" />
       <limit
-        lower="-3.14"
-        upper="3.14"
+        lower="-6.28"
+        upper="6.28"
         effort="0"
         velocity="0" />
@@ -412,6 +412,6 @@
         xyz="0 0 1" />
       <limit
-        lower="-3.14"
-        upper="3.14"
+        lower="-6.28"
+        upper="6.28"
         effort="0"
         velocity="0" />
@@ -426,6 +426,6 @@
         xyz="0 0 -1" />
       <limit
-        lower="-3.14"
-        upper="3.14"
+        lower="-6.28"
+        upper="6.28"
         effort="0"
         velocity="0" />
@@ -440,6 +440,6 @@
         xyz="0 1 0" />
       <limit
-        lower="-3.14"
-        upper="3.14"
+        lower="-6.28"
+        upper="6.28"
         effort="0"
         velocity="0" />
@@ -468,5 +468,5 @@
     <joint name="${prefix}flange-tool0" type="fixed">
       <!-- default toolframe: X+ left, Y+ up, Z+ front -->
-      <origin xyz="0 0 0" rpy="${pi/2.0} 0 ${pi/2.0}"/>
+      <origin xyz="0 0 -0.1" rpy="${pi/2.0} 0 ${pi/2.0}"/>
       <parent link="${prefix}flange"/>
       <child link="${prefix}tool0"/>
