Commit message: Arm configuration finally looks good

File: ur_description/urdf/ur_macro.xacro (robot description, xacro)
@@ -68,23 +68,146 @@
       <inertial>
         <origin
-          xyz="0 0 0.014753"
-          rpy="0 0 0" />
-        <mass
-          value="0.82586" />
-        <inertia
-          ixx="0.0020803"
-          ixy="1.735E-19"
-          ixz="3.2973E-19"
-          iyy="0.0020803"
-          iyz="3.6808E-19"
-          izz="0.0039193" />
-      </inertial>
-      <visual>
-        <origin
-          xyz="0 0 0"
-          rpy="0 0 0" />
-        <geometry>
-          <mesh
-            filename="package://al_arm_5_2/meshes/base.STL" />
+          xyz="0.0014629 -2.6906E-07 0.012448"
+          rpy="0 0 0" />
+        <mass
+          value="1.5303" />
+        <inertia
+          ixx="0.0048294"
+          ixy="-7.7706E-08"
+          ixz="1.2591E-05"
+          iyy="0.0048663"
+          iyz="1.1079E-08"
+          izz="0.0094303" />
+      </inertial>
+      <visual>
+        <origin
+          xyz="0 0 0"
+          rpy="0 0 0" />
+        <geometry>
+          <mesh
+            filename="package://al_arm_2_5/meshes/base_link.STL" />
+        </geometry>
+        <material
+          name="">
+          <color
+            rgba="0.89804 0.91765 0.92941 1" />
+        </material>
+      </visual>
+<!--
+      <collision>
+        <origin
+          xyz="0 0 0"
+          rpy="0 0 0" />
+        <geometry>
+          <mesh
+            filename="package://al_arm_2_5/meshes/base_link.STL" />
+        </geometry>
+      </collision>
+-->
+    </link>
+    <link name="${prefix}shoulder_link">
+      <inertial>
+        <origin
+          xyz="-0.011994 0.0070501 0.079805"
+          rpy="0 0 0" />
+        <mass
+          value="1.2061" />
+        <inertia
+          ixx="0.0043639"
+          ixy="0.00024188"
+          ixz="-1.4432E-05"
+          iyy="0.0046436"
+          iyz="7.8064E-06"
+          izz="0.0045073" />
+      </inertial>
+      <visual>
+        <origin
+          xyz="0 0 0"
+          rpy="0 0 0" />
+        <geometry>
+          <mesh
+            filename="package://al_arm_2_5/meshes/link_1.STL" />
+        </geometry>
+        <material
+          name="">
+          <color
+            rgba="0.89804 0.91765 0.92941 1" />
+        </material>
+      </visual>
+<!--
+      <collision>
+        <origin
+          xyz="0 0 0"
+          rpy="0 0 0" />
+        <geometry>
+          <mesh
+            filename="package://al_arm_2_5/meshes/link_1.STL" />
+        </geometry>
+      </collision>
+-->
+    </link>
+    <link name="${prefix}upper_arm_link">
+      <inertial>
+        <origin
+          xyz="0.16523 0.091649 0.083369"
+          rpy="0 0 0" />
+        <mass
+          value="2.3874" />
+        <inertia
+          ixx="0.0084074"
+          ixy="-0.0010604"
+          ixz="-7.337E-08"
+          iyy="0.0097311"
+          iyz="1.4278E-07"
+          izz="0.009462" />
+      </inertial>
+      <visual>
+        <origin
+          xyz="0 0 0"
+          rpy="0 0 0" />
+        <geometry>
+          <mesh
+            filename="package://al_arm_2_5/meshes/link_2.STL" />
+        </geometry>
+        <material
+          name="">
+          <color
+            rgba="0.89804 0.91765 0.92941 1" />
+        </material>
+      </visual>
+<!--
+      <collision>
+        <origin
+          xyz="0 0 0"
+          rpy="0 0 0" />
+        <geometry>
+          <mesh
+            filename="package://al_arm_2_5/meshes/link_2.STL" />
+        </geometry>
+      </collision>
+-->
+    </link>
+    <link name="${prefix}forearm_link">
+      <inertial>
+        <origin
+          xyz="0.046835 0.11058 0.082124"
+          rpy="0 0 0" />
+        <mass
+          value="1.3594" />
+        <inertia
+          ixx="0.0033204"
+          ixy="-0.00013061"
+          ixz="-9.2169E-06"
+          iyy="0.0033902"
+          iyz="-2.5688E-05"
+          izz="0.0036184" />
+      </inertial>
+      <visual>
+        <origin
+          xyz="0 0 0"
+          rpy="0 0 0" />
+        <geometry>
+          <mesh
+            filename="package://al_arm_2_5/meshes/link_3.STL" />
         </geometry>
         <material
@@ -101,113 +224,31 @@
         <geometry>
           <mesh
-            filename="package://al_arm_5_2/meshes/base.STL" />
-        </geometry>
-      </collision>
--->
-    </link>
-    <link name="${prefix}shoulder_link">
-      <inertial>
-        <origin
-          xyz="0.0057811 -4.7696E-10 0.086487"
-          rpy="0 0 3.141" />
-        <mass
-          value="2.207" />
-        <inertia
-          ixx="0.0095841"
-          ixy="8.9967E-10"
-          ixz="-0.0003"
-          iyy="0.0097275"
-          iyz="4.4737E-10"
-          izz="0.0055768" />
-      </inertial>
-      <visual>
-        <origin
-          xyz="0 0 0"
-          rpy="0 0 3.141" />
-        <geometry>
-          <mesh
-            filename="package://al_arm_5_2/meshes/seg1.STL" />
-        </geometry>
-        <material
-          name="">
-          <color
-            rgba="0.50196 0.50196 1 1" />
-        </material>
-      </visual>
-<!--
-      <collision>
-        <origin
-          xyz="0 0 0"
-          rpy="0 0 0" />
-        <geometry>
-          <mesh
-            filename="package://al_arm_5_2/meshes/seg1.STL" />
-        </geometry>
-      </collision>
--->
-    </link>
-    <link name="${prefix}upper_arm_link">
-      <inertial>
-        <origin
-          xyz="0.6 0.0005672 0.085941"
-          rpy="0 0 0" />
-        <mass
-          value="2.1" />
-        <inertia
-          ixx="0.0096686"
-          ixy="-1.7798E-05"
-          ixz="-2.2764E-05"
-          iyy="0.0097485"
-          iyz="-4.8304E-06"
-          izz="0.0051536" />
-      </inertial>
-      <visual>
-        <origin
-          xyz="0 0 0"
-          rpy="0 0 0" />
-        <geometry>
-          <mesh
-            filename="package://al_arm_5_2/meshes/seg2.STL" />
-        </geometry>
-        <material
-          name="">
-          <color
-            rgba="0.50196 0.50196 1 1" />
-        </material>
-      </visual>
-<!--
-      <collision>
-        <origin
-          xyz="0 0 0"
-          rpy="0 0 0" />
-        <geometry>
-          <mesh
-            filename="package://al_arm_5_2/meshes/seg2.STL" />
-        </geometry>
-      </collision>
--->
-    </link>
-    <link name="${prefix}forearm_link">
-      <inertial>
-        <origin
-          xyz="-5.0864E-07 0.0083839 0.20092"
-          rpy="0 0 0" />
-        <mass
-          value="0.81968" />
-        <inertia
-          ixx="0.0025453"
-          ixy="-5.2922E-10"
-          ixz="-3.0369E-10"
-          iyy="0.0016077"
-          iyz="-0.00011692"
-          izz="0.0019806" />
-      </inertial>
-      <visual>
-        <origin
-          xyz="0 0 0"
-          rpy="0 0 0" />
-        <geometry>
-          <mesh
-            filename="package://al_arm_5_2/meshes/seg3.STL" />
+            filename="package://al_arm_2_5/meshes/link_3.STL" />
+        </geometry>
+      </collision>
+-->
+    </link>
+    <link name="${prefix}wrist_1_link">
+      <inertial>
+        <origin
+          xyz="-0.0028354 1.2239E-06 0.055457"
+          rpy="0 0 0" />
+        <mass
+          value="0.78328" />
+        <inertia
+          ixx="0.0020107"
+          ixy="-2.0341E-07"
+          ixz="-3.1182E-05"
+          iyy="0.0022157"
+          iyz="-2.3219E-08"
+          izz="0.0017318" />
+      </inertial>
+      <visual>
+        <origin
+          xyz="0 0 0"
+          rpy="0 0 0" />
+        <geometry>
+          <mesh
+            filename="package://al_arm_2_5/meshes/link_4.STL" />
         </geometry>
         <material
@@ -224,46 +265,5 @@
         <geometry>
           <mesh
-            filename="package://al_arm_5_2/meshes/seg3.STL" />
-        </geometry>
-      </collision>
--->
-    </link>
-    <link name="${prefix}wrist_1_link">
-      <inertial>
-        <origin
-          xyz="0.028904 -0.03325 0.050924"
-          rpy="0 0 0" />
-        <mass
-          value="1.5416" />
-        <inertia
-          ixx="0.0025041"
-          ixy="0.00055564"
-          ixz="-0.00017823"
-          iyy="0.0023479"
-          iyz="0.00020503"
-          izz="0.0028189" />
-      </inertial>
-      <visual>
-        <origin
-          xyz="0 0 0"
-          rpy="0 0 0" />
-        <geometry>
-          <mesh
-            filename="package://al_arm_5_2/meshes/seg4.STL" />
-        </geometry>
-        <material
-          name="">
-          <color
-            rgba="0.50196 0.50196 1 1" />
-        </material>
-      </visual>
-<!--
-      <collision>
-        <origin
-          xyz="0 0 0"
-          rpy="0 0 0" />
-        <geometry>
-          <mesh
-            filename="package://al_arm_5_2/meshes/seg4.STL" />
+            filename="package://al_arm_2_5/meshes/link_4.STL" />
         </geometry>
       </collision>
@@ -273,38 +273,38 @@
       <inertial>
         <origin
-          xyz="5.2201E-07 -0.003931 0.039853"
-          rpy="0 0 0" />
-        <mass
-          value="0.71921" />
-        <inertia
-          ixx="0.0019666"
-          ixy="-3.0762E-10"
-          ixz="1.656E-11"
-          iyy="0.0010669"
-          iyz="5.6958E-05"
-          izz="0.0017541" />
-      </inertial>
-      <visual>
-        <origin
-          xyz="0 0 0"
-          rpy="0 0 0" />
-        <geometry>
-          <mesh
-            filename="package://al_arm_5_2/meshes/seg5.STL" />
-        </geometry>
-        <material
-          name="">
-          <color
-            rgba="0.50196 0.50196 1 1" />
-        </material>
-      </visual>
-<!--
-      <collision>
-        <origin
-          xyz="0 0 0"
-          rpy="0 0 0" />
-        <geometry>
-          <mesh
-            filename="package://al_arm_5_2/meshes/seg5.STL" />
+          xyz="0.00029676 0.0028204 0.055458"
+          rpy="0 0 0" />
+        <mass
+          value="0.78327" />
+        <inertia
+          ixx="0.0022136"
+          ixy="-2.1109E-05"
+          ixz="3.2374E-06"
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
Commit message: Increase joint limits

File: ur_description/urdf/ur_macro.xacro (robot description, xacro)
@@ -372,6 +372,6 @@
         xyz="0 0 1" />
       <limit
-        lower="3.15"
-        upper="-3.15"
+        lower="-6.28"
+        upper="6.28"
         effort="0"
         velocity="0" />
@@ -386,6 +386,6 @@
         xyz="0 0 1" />
       <limit
-        lower="3.15"
-        upper="-3.15"
+        lower="-6.28"
+        upper="6.28"
         effort="0"
         velocity="0" />
@@ -400,6 +400,6 @@
         xyz="0 0 -1" />
       <limit
-        lower="3.15"
-        upper="-3.15"
+        lower="-6.28"
+        upper="6.28"
         effort="0"
         velocity="0" />
@@ -414,6 +414,6 @@
         xyz="0 0 -1" />
       <limit
-        lower="3.15"
-        upper="-3.15"
+        lower="-6.28"
+        upper="6.28"
         effort="0"
         velocity="0" />
@@ -442,6 +442,6 @@
         xyz="0 -0.10453 -0.99452" />
       <limit
-        lower="3.15"
-        upper="-3.15"
+        lower="-6.28"
+        upper="6.28"
         effort="0"
         velocity="0" />
@@ -470,5 +470,5 @@
     <joint name="${prefix}flange-tool0" type="fixed">
       <!-- default toolframe: X+ left, Y+ up, Z+ front -->
-      <origin xyz="0 0 -0.1" rpy="${pi/2.0} 0 ${pi/2.0}"/>
+      <origin xyz="0 0 0" rpy="${pi/2.0} 0 ${pi/2.0}"/>
       <parent link="${prefix}flange"/>
       <child link="${prefix}tool0"/>
